Commit message: Added VLP16 model and proper frames

File: urdf/clem_description.urdf.xacro (robot description, xacro)
@@ -2,9 +2,21 @@
 <robot xmlns:xacro="http://www.ros.org/wiki/xacro">
 <!-- This Is A Link -->
+	<link name="velodyne_mount" >
+<visual>
+		<geometry>
+			<mesh filename="package://clem_description/meshes/VLP16.dae"/>
+		</geometry>
+	</visual>
+</link>
+	<joint name="velodyne_mount_joint" type="fixed" >
+	 <parent link="mid_mount" />
+	 <child link="velodyne_mount" />
+	 <origin xyz="0 0 0.1" rpy="0 0 0" />
+	</joint>
 	<link name="velodyne" />
 	<joint name="velodyne_joint" type="fixed" >
-	 <parent link="mid_mount" />
+	 <parent link="velodyne_mount" />
 	 <child link="velodyne" />
-	 <origin xyz="0 0 0.1" rpy="0 0 0" />
+	 <origin xyz="0 0 0.0378" rpy="0 0 0" />
 	</joint>
 </robot>
